Commit message: fixed frame update

File: src/urdfs/hubo_description.urdf (robot description, URDF)
Before this commit: robot DRC_HUBO, 63 links, 62 joints
Joints:
- joint LEFT_ELBOW: limit lower=-2.96705972839036 upper=0.8726646259971648 effort=100000 velocity=7.644542123735163 -> lower=-2.96705972839036 upper=-0.5 effort=100000 velocity=7.644542123735163
- joint LEFT_SHOULDER_YAW: limit lower=-2.96705972839036 upper=2.96705972839036 effort=100000 velocity=7.644542123735163 -> lower=-2.2 upper=2.2 effort=100000 velocity=7.644542123735163
- joint RIGHT_ELBOW: limit lower=-2.96705972839036 upper=0.8726646259971648 effort=100000 velocity=7.644542123735163 -> lower=-2.96705972839036 upper=-0.5 effort=100000 velocity=7.644542123735163
- joint RIGHT_SHOULDER_YAW: limit lower=-2.96705972839036 upper=2.96705972839036 effort=100000 velocity=7.644542123735163 -> lower=-2.2 upper=2.2 effort=100000 velocity=7.644542123735163
