Commit message: updated gitignore

File: src/RelaxedIK/urdfs/hubo_description.urdf (robot description, URDF)
Before this commit: robot DRC_HUBO, 63 links, 62 joints
Joints:
- joint RIGHT_SHOULDER_ROLL: limit lower=-0.5235987755982988 upper=3.6651914291880923 effort=100000 velocity=4.254240051736178 -> lower=-3.6651914291880923 upper=0.52 effort=100000 velocity=4.254240051736178

Commit message: updated urdf

File: src/RelaxedIK/urdfs/hubo_description.urdf (robot description, URDF)
Before this commit: robot DRC_HUBO, 63 links, 62 joints
Joints:
- joint LEFT_SHOULDER_PITCH: limit lower=-1.3962634015954636 upper=4.537856055185257 effort=100000 velocity=4.254240051736178 -> lower=-4.537856055185257 upper=1.3962634015954636 effort=100000 velocity=4.254240051736178
- joint RIGHT_SHOULDER_PITCH: limit lower=-1.3962634015954636 upper=4.537856055185257 effort=100000 velocity=4.254240051736178 -> lower=-4.537856055185257 upper=1.3962634015954636 effort=100000 velocity=4.254240051736178
- joint WAIST: limit lower=-6.1086523819801535 upper=6.1086523819801535 effort=100000 velocity=2.0 -> lower=-1.0 upper=1.0 effort=100000 velocity=2.0
