Commit message: more camera stuff

File: src/RelaxedIK/urdfs/jaco7_pair.urdf (robot description, URDF)
Before this commit: robot j2s7s300, 33 links, 32 joints
Joints:
- joint connect_root_and_world_b: origin xyz=0 0.8 0 rpy=0 0 0 -> xyz=0 0.4 0 rpy=0 0 0

Commit message: support for visual exploration

File: src/RelaxedIK/urdfs/jaco7_pair.urdf (robot description, URDF)
Before this commit: robot j2s7s300, 33 links, 32 joints
Joints:
- joint connect_root_and_world_b: origin xyz=0 0.4 0 rpy=0 0 0 -> xyz=0 0.4 0.0 rpy=0 0 0

Commit message: switched robots

File: src/RelaxedIK/urdfs/jaco7_pair.urdf (robot description, URDF)
Before this commit: robot j2s7s300, 33 links, 32 joints
Joints:
- joint connect_root_and_world_b: origin xyz=0 0.4 0.0 rpy=0 0 0 -> xyz=-0.1905 0.4 0.0 rpy=0 0 0
