Commit message: subscriber classes

File: src/RelaxedIK/urdfs/hubo_description2.urdf (robot description, URDF)
Before this commit: robot DRC_HUBO, 63 links, 62 joints
Joints:
- removed joint WAIST2
- added joint base_footprint_joint: type fixed, parent base_footprint, child Body_TORSO, origin xyz=0 0 0 rpy=0 0 0
