Commit message: fixed bug related to movo robot

File: src/RelaxedIK/urdfs/sawyer.urdf (robot description, URDF)
Before this commit: robot sawyer, 24 links, 23 joints
Links:
- link controller_box: geometry collision mesh filename=file:///tmp/controller_box_mesh.dae scale=1 1 1; visual mesh filename=file:///tmp/controller_box_mesh.dae scale=1 1 1
- link head: geometry collision mesh filename=file:///tmp/head_mesh.dae scale=1 1 1; visual mesh filename=file:///tmp/head_mesh.dae scale=1 1 1
- link pedestal: mass 60.86397744 -> 60.864; geometry collision mesh filename=file:///tmp/pedestal_mesh.dae scale=1 1 1; visual mesh filename=file:///tmp/pedestal_mesh.dae scale=1 1 1
- link pedestal_feet: geometry collision mesh filename=file:///tmp/pedestal_feet_mesh.dae scale=1 1 1; visual mesh filename=file:///tmp/pedestal_feet_mesh.dae scale=1 1 1
- link right_arm_base_link: geometry collision mesh filename=file:///tmp/right_arm_base_link_mesh.dae scale=1 1 1; visual mesh filename=file:///tmp/right_arm_base_link_mesh.dae scale=1 1 1
- link right_hand: mass 1.0E-08 -> 1e-08; geometry collision mesh filename=file:///tmp/right_hand_mesh.dae scale=1 1 1; visual mesh filename=file:///tmp/right_hand_mesh.dae scale=1 1 1
- link right_l0: geometry collision mesh filename=file:///tmp/right_l0_mesh.dae scale=1 1 1; visual mesh filename=file:///tmp/right_l0_mesh.dae scale=1 1 1
- link right_l1: geometry collision mesh filename=file:///tmp/right_l1_mesh.dae scale=1 1 1; visual mesh filename=file:///tmp/right_l1_mesh.dae scale=1 1 1
- link right_l1_2: mass 1.0E-08 -> 1e-08; geometry collision mesh filename=file:///tmp/right_l1_2_mesh.dae scale=1 1 1; visual mesh filename=file:///tmp/right_l1_2_mesh.dae scale=1 1 1
- link right_l2: geometry collision mesh filename=file:///tmp/right_l2_mesh.dae scale=1 1 1; visual mesh filename=file:///tmp/right_l2_mesh.dae scale=1 1 1
- link right_l2_2: mass 1.0E-08 -> 1e-08; geometry collision mesh filename=file:///tmp/right_l2_2_mesh.dae scale=1 1 1; visual mesh filename=file:///tmp/right_l2_2_mesh.dae scale=1 1 1
- link right_l3: geometry collision mesh filename=file:///tmp/right_l3_mesh.dae scale=1 1 1; visual mesh filename=file:///tmp/right_l3_mesh.dae scale=1 1 1
- link right_l4: geometry collision mesh filename=file:///tmp/right_l4_mesh.dae scale=1 1 1; visual mesh filename=file:///tmp/right_l4_mesh.dae scale=1 1 1
- link right_l4_2: mass 1.0E-08 -> 1e-08; geometry collision mesh filename=file:///tmp/right_l4_2_mesh.dae scale=1 1 1; visual mesh filename=file:///tmp/right_l4_2_mesh.dae scale=1 1 1
- link right_l5: geometry collision mesh filename=file:///tmp/right_l5_mesh.dae scale=1 1 1; visual mesh filename=file:///tmp/right_l5_mesh.dae scale=1 1 1
- link right_l6: geometry collision mesh filename=file:///tmp/right_l6_mesh.dae scale=1 1 1; visual mesh filename=file:///tmp/right_l6_mesh.dae scale=1 1 1
- link screen: geometry collision mesh filename=file:///tmp/screen_mesh.dae scale=1 1 1; visual mesh filename=file:///tmp/screen_mesh.dae scale=1 1 1
- link torso: geometry collision mesh filename=file:///tmp/torso_mesh.dae scale=1 1 1; visual mesh filename=file:///tmp/torso_mesh.dae scale=1 1 1
Joints:
- joint controller_box_fixed: axis (none) -> 0 0 0; limit (none) -> lower=0 upper=0 effort=100 velocity=0.5; origin xyz=0.0 0.0 0.0 rpy=0 0 0 -> xyz=0 0 0 rpy=0 -0 0 
- joint display_joint: axis (none) -> 0 0 0; limit (none) -> lower=0 upper=0 effort=100 velocity=0.5; origin xyz=0.03 0.0 0.105 rpy=1.57079632679 0 1.57079632679 -> xyz=0.03 0 0.105 rpy=1.5708 -3.33067e-16 1.5708 
- joint head_camera: limit (none) -> lower=0 upper=0 effort=100 velocity=0.5; origin xyz=0.0228027 0 0.216572 rpy=-2.1293 0 -1.57079632679 -> xyz=0.0228027 0 0.216572 rpy=-2.1293 -6.10623e-16 -1.5708 
- joint head_pan: origin xyz=0 0 0.2965 rpy=0 0 0 -> xyz=0 0 0.2965 rpy=0 -0 0 
- joint pedestal_feet_fixed: axis (none) -> 0 0 0; limit (none) -> lower=0 upper=0 effort=100 velocity=0.5; origin xyz=0.0 0.0 0.0 rpy=0 0 0 -> xyz=0 0 0 rpy=0 -0 0 
- joint pedestal_fixed: axis (none) -> 0 0 0; limit (none) -> lower=0 upper=0 effort=100 velocity=0.5; origin xyz=0.0 0.0 0.0 rpy=0 0 0 -> xyz=0 0 0 rpy=0 -0 0 
- joint right_arm_itb: axis 0 0 1 -> 0 0 0; limit (none) -> lower=0 upper=0 effort=100 velocity=0.5; origin xyz=-.055 0 .075 rpy=0 -1.57079632679 0 -> xyz=-0.055 0 0.075 rpy=0 -1.5708 0 
- joint right_arm_mount: axis (none) -> 0 0 0; limit (none) -> lower=0 upper=0 effort=100 velocity=0.5; origin xyz=0.0 0.0 0.0 rpy=0 0 0 -> xyz=0 0 0 rpy=0 -0 0 
- joint right_hand: axis 0 0 1 -> 0 0 0; limit (none) -> lower=0 upper=0 effort=100 velocity=0.5; origin xyz=0 0 0.0245 rpy=0 0 1.570796 -> xyz=0 0 0.0245 rpy=0 -0 1.5708 
- joint right_hand_camera: limit (none) -> lower=0 upper=0 effort=100 velocity=0.5; origin xyz=0.039552 -0.033 0.0695 rpy=0 1.57079632679 0 -> xyz=0.039552 -0.033 0.0695 rpy=0 1.5708 -0 
- joint right_j0: limit lower=-3.0503 upper=3.0503 effort=80.0 velocity=1.74 -> lower=-3.0503 upper=3.0503 effort=80 velocity=1.74; origin xyz=0 0 0.08 rpy=0 0 0 -> xyz=0 0 0.08 rpy=0 -0 0 
- joint right_j1: limit lower=-3.8095 upper=2.2736 effort=80.0 velocity=1.328 -> lower=-3.8095 upper=2.2736 effort=80 velocity=1.328; origin xyz=0.081 0.05 0.237 rpy=-1.57079632679 1.57079632679 0 -> xyz=0.081 0.05 0.237 rpy=0 1.5708 1.5708 
- joint right_j1_2: axis 0 0 1 -> 0 0 0; limit (none) -> lower=0 upper=0 effort=100 velocity=0.5; origin xyz=0 0 0 rpy=0 0 0 -> xyz=0 0 0 rpy=0 -0 0 
- joint right_j2: limit lower=-3.0426 upper=3.0426 effort=40.0 velocity=1.957 -> lower=-3.0426 upper=3.0426 effort=40 velocity=1.957; origin xyz=0 -0.14 0.1425 rpy=1.57079632679 0 0 -> xyz=0 -0.14 0.1425 rpy=1.5708 -0 0 
- joint right_j2_2: axis 0 0 1 -> 0 0 0; limit (none) -> lower=0 upper=0 effort=100 velocity=0.5; origin xyz=0 0 0 rpy=0 0 0 -> xyz=0 0 0 rpy=0 -0 0 
- joint right_j3: limit lower=-3.0439 upper=3.0439 effort=40.0 velocity=1.957 -> lower=-3.0439 upper=3.0439 effort=40 velocity=1.957; origin xyz=0 -0.042 0.26 rpy=-1.57079632679 0 0 -> xyz=0 -0.042 0.26 rpy=-1.5708 0 0 
- joint right_j4: limit lower=-2.9761 upper=2.9761 effort=9.0 velocity=3.485 -> lower=-2.9761 upper=2.9761 effort=9 velocity=3.485; origin xyz=0 -0.125 -0.1265 rpy=1.57079632679 0 0 -> xyz=0 -0.125 -0.1265 rpy=1.5708 -0 0 
- joint right_j4_2: axis 0 0 1 -> 0 0 0; limit (none) -> lower=0 upper=0 effort=100 velocity=0.5; origin xyz=0 0 0 rpy=0 0 0 -> xyz=0 0 0 rpy=0 -0 0 
- joint right_j5: limit lower=-2.9761 upper=2.9761 effort=9.0 velocity=3.485 -> lower=-2.9761 upper=2.9761 effort=9 velocity=3.485; origin xyz=0 0.031 0.275 rpy=-1.57079632679 0 0 -> xyz=0 0.031 0.275 rpy=-1.5708 0 0 
- joint right_j6: limit lower=-4.7124 upper=4.7124 effort=9.0 velocity=4.545 -> lower=-4.7124 upper=4.7124 effort=9 velocity=4.545; origin xyz=0 -0.11 0.1053 rpy=-1.57079632679 -0.17453 3.1416 -> xyz=0 -0.11 0.1053 rpy=-1.5708 -0.17453 -3.14159 
- joint right_torso_itb: axis 0 0 1 -> 0 0 0; limit (none) -> lower=0 upper=0 effort=100 velocity=0.5; origin xyz=-.055 0 .22 rpy=0 -1.57079632679 0 -> xyz=-0.055 0 0.22 rpy=0 -1.5708 0 
- joint right_wrist: limit (none) -> lower=0 upper=0 effort=100 velocity=0.5; origin xyz=0 0 0.10541 rpy=1.57079632679 0 0 -> xyz=0 0 0.10541 rpy=1.5708 -0 0 
- joint torso_t0: axis (none) -> 0 0 0; limit (none) -> lower=0 upper=0 effort=100 velocity=0.5; origin xyz=0 0 0 rpy=0 0 0 -> xyz=0 0 0 rpy=0 -0 0 
